Commit message: Include gazebo materials

File: axebot_description/urdf/axebot_description.urdf.xacro (robot description, xacro)
@@ -15,4 +15,5 @@
     <xacro:property name="distance_to_chassis" value="0.0025"/>
     <xacro:include filename="$(find axebot_description)/urdf/axebot_wheels.urdf.xacro"/>
+    <xacro:include filename="$(find axebot_description)/urdf/axebot_materials.xacro"/>
     <xacro:macro name="axebot" params="prefix">
         <link name="${prefix}base_link">
@@ -22,5 +23,5 @@
                     <cylinder radius="${base_radius}" length="${base_height}"/>
                 </geometry>
-                <material name="orange"/>
+                <material name="black"/>
             </visual>
         </link>

File: axebot_description/urdf/axebot_wheels.urdf.xacro (robot description, xacro)
@@ -14,4 +14,5 @@
                     <cylinder radius="${wheel_shaft_radius}" length="${distance_to_chassis}"/>
                 </geometry>
+                <material name="grey"/>
             </visual>
         </link>
@@ -28,4 +29,5 @@
                     <cylinder radius="${wheel_radius}" length="${wheel_thickness}"/>
                 </geometry>
+                <material name="green"/>
             </visual>
         </link>

Commit message: Add inertia and collision properties

File: axebot_description/urdf/axebot_description.urdf.xacro (robot description, xacro)
@@ -6,12 +6,13 @@
     <xacro:property name="base_height" value="0.04"/>
     <xacro:property name="robot_height" value="0.053"/>
-    <xacro:property name="wheel_mass" value="0.3" />
+    <xacro:property name="wheel_mass" value="0.268" />
     <xacro:property name="wheel_radius" value="0.05" />
     <xacro:property name="wheel_shaft_radius" value="0.005" />
+    <xacro:property name="shaft_mass" value="0.01" />
     <!-- The sum of the base radius, half of wheel thickness, and the shat
     length must be equal the robot radius L = 0.1 m used in the kinematic model -->
     <xacro:property name="base_radius" value="0.085"/>
     <xacro:property name="wheel_thickness" value="0.025" />
-    <xacro:property name="distance_to_chassis" value="0.0025"/>
+    <xacro:property name="shaft_length" value="0.0025"/>
     <xacro:include filename="$(find axebot_description)/urdf/axebot_wheels.urdf.xacro"/>
     <xacro:include filename="$(find axebot_description)/urdf/axebot_materials.xacro"/>
@@ -25,4 +26,14 @@
                 <material name="black"/>
             </visual>
+            <collision>
+                <origin xyz="0.0 0.0 ${robot_height}" rpy="0.0 0.0 0.0"/>
+                <geometry>
+                    <cylinder radius="${base_radius}" length="${base_height}"/>
+                </geometry>
+                <material name="black"/>
+            </collision>
+            <xacro:inertial_cylinder mass="${base_mass}" radius="${base_radius}" length="${base_height}">
+                <origin xyz="0.0 0.0 ${robot_height}" rpy="0.0 0.0 0.0"/>
+            </xacro:inertial_cylinder>
         </link>
         <xacro:wheel prefix="${prefix}" num="1" theta="${PI}"/>

File: axebot_description/urdf/axebot_wheels.urdf.xacro (robot description, xacro)
@@ -1,4 +1,17 @@
 <?xml version="1.0"?>
 <robot xmlns:xacro="http://www.ros.org/wiki/xacro">
+    <xacro:macro name="inertial_cylinder" params="mass length radius *origin">
+        <inertial>
+            <xacro:insert_block name="origin"/>
+            <mass value="${mass}" />
+            <inertia
+                ixx="${(1/12) * mass * (3*radius*radius + length*length)}"
+                ixy="0.0"
+                ixz="0.0"
+                iyy="${(1/12) * mass * (3*radius*radius + length*length)}"
+                iyz="0.0"
+                izz="${(1/2) * mass * (radius*radius)}" />
+            </inertial>
+    </xacro:macro>
     <xacro:macro name="wheel" params="prefix num theta">
         <joint name="${prefix}wheel${num}_shaft_joint" type="fixed">
@@ -6,17 +19,25 @@
             <parent link="${prefix}base_link"/>
             <child link="${prefix}wheel${num}_shaft_link"/>
-            <axis xyz="${base_radius} 0.0 0.0"/>
         </joint>
         <link name="${prefix}wheel${num}_shaft_link">
             <visual>
-                <origin xyz="0.0 0.0 -${distance_to_chassis/2}" rpy="0.0 0.0 0.0"/>
+                <origin xyz="0.0 0.0 -${shaft_length/2}" rpy="0.0 0.0 0.0"/>
                 <geometry>
-                    <cylinder radius="${wheel_shaft_radius}" length="${distance_to_chassis}"/>
+                    <cylinder radius="${wheel_shaft_radius}" length="${shaft_length}"/>
                 </geometry>
                 <material name="grey"/>
             </visual>
+            <collision>
+                <origin xyz="0.0 0.0 -${shaft_length/2}" rpy="0.0 0.0 0.0"/>
+                <geometry>
+                    <cylinder radius="${wheel_shaft_radius}" length="${shaft_length}"/>
+                </geometry>
+            </collision>
+            <xacro:inertial_cylinder mass="${shaft_mass}" radius="${wheel_shaft_radius}" length="${shaft_length}">
+                <origin xyz="0.0 0.0 -${shaft_length/2}" rpy="0.0 0.0 0.0"/>
+            </xacro:inertial_cylinder>
         </link>
         <joint name="${prefix}wheel${num}_joint" type="continuous">
-            <origin xyz="0.0 0.0 -${distance_to_chassis}" rpy="0.0 0.0 0.0"/>
+            <origin xyz="0.0 0.0 -${shaft_length}" rpy="0.0 0.0 0.0"/>
             <parent link="${prefix}wheel${num}_shaft_link"/>
             <child link="${prefix}wheel${num}_link"/>
@@ -31,4 +52,13 @@
                 <material name="green"/>
             </visual>
+            <collision>
+                <origin xyz="0.0 0.0 -${wheel_thickness/2}" rpy="0.0 0.0 0.0"/>
+                <geometry>
+                    <cylinder radius="${wheel_radius}" length="${wheel_thickness}"/>
+                </geometry>
+            </collision>
+            <xacro:inertial_cylinder mass="${wheel_mass}" radius="${wheel_radius}" length="${wheel_thickness}">
+                <origin xyz="0.0 0.0 -${wheel_thickness/2}" rpy="0.0 0.0 0.0"/>
+            </xacro:inertial_cylinder>
         </link>
     </xacro:macro>
