Commit message: Add real omnidirectional wheel

File: axebot_description/urdf/gazebo.urdf.xacro (robot description, xacro)
@@ -4,15 +4,15 @@
     </gazebo>
     <gazebo reference="wheel1_link">
-        <material>Gazebo/Green</material>
+        <material>Gazebo/Grey</material>
         <mu1>0.2</mu1>
         <mu2>0.2</mu2>
     </gazebo>
     <gazebo reference="wheel2_link">
-        <material>Gazebo/Green</material>
+        <material>Gazebo/Grey</material>
         <mu1>0.2</mu1>
         <mu2>0.2</mu2>
     </gazebo>
     <gazebo reference="wheel3_link">
-        <material>Gazebo/Green</material>
+        <material>Gazebo/Grey</material>
         <mu1>0.2</mu1>
         <mu2>0.2</mu2>

File: axebot_description/urdf/wheel.urdf.xacro (robot description, xacro)
@@ -1,4 +1,5 @@
 <?xml version="1.0"?>
 <robot xmlns:xacro="http://www.ros.org/wiki/xacro">
+    <xacro:property name="distance_to_roller_center" value="0.04645"/>
     <xacro:macro name="inertial_cylinder" params="mass length radius *origin">
         <inertial>
@@ -13,4 +14,37 @@
                 izz="${(1/2) * mass * (radius*radius)}" />
             </inertial>
+    </xacro:macro>
+    <xacro:macro name="insert_roller" params="parent reflect theta suffix wheel">
+        <joint name="rim_to_roller${wheel}${suffix}joint" type="fixed">
+            <origin xyz="${distance_to_roller_center*cos(theta)} ${distance_to_roller_center*sin(theta)} ${reflect*0.008}" rpy="0.0 0.0 ${theta-PI/2}"/>
+            <parent link="${parent}"/>
+            <child link="roller${wheel}${suffix}_link"/>
+            <axis xyz="1.0 0.0 0.0"/>
+        </joint>
+        <link name="roller${wheel}${suffix}_link">
+            <visual>
+                <origin xyz="0.0 0.0 0.0" rpy="0.0 0.0 0.0"/>
+                <geometry>
+                    <mesh filename="file://$(find axebot_description)/meshes/roller.stl"/>
+                </geometry>
+                <material name="green"/>
+            </visual>
+            <collision>
+                <origin xyz="0.0 0.0 0.0" rpy="0.0 0.0 0.0"/>
+                <geometry>
+                    <mesh filename="file://$(find axebot_description)/meshes/roller.stl"/>
+                </geometry>
+            </collision>
+            <inertial>
+                <origin xyz="0.0 0.0 0.0" rpy="0.0 0.0 0.0"/>
+                <mass value="0.003"/>
+                <inertia ixx="5.3e-8"
+                         ixy="0.0"
+                         ixz="0.0"
+                         iyy="7.6e-8"
+                         iyz="0.0"
+                         izz="7.6e-8"/>
+            </inertial>
+        </link>
     </xacro:macro>
     <xacro:macro name="wheel" params="parent suffix theta">
@@ -46,9 +80,9 @@
         <link name="wheel${suffix}_link">
             <visual>
-                <origin xyz="0.0 0.0 -${wheel_thickness/2}" rpy="0.0 0.0 0.0"/>
+                <origin xyz="0.0 0.0 0.0" rpy="0.0 0.0 0.0"/>
                 <geometry>
-                    <cylinder radius="${wheel_radius}" length="${wheel_thickness}"/>
+                    <mesh filename="file://$(find axebot_description)/meshes/rim.stl"/>
                 </geometry>
-                <material name="green"/>
+                <material name="grey"/>
             </visual>
             <collision>
@@ -58,8 +92,39 @@
                 </geometry>
             </collision>
-            <xacro:inertial_cylinder mass="${wheel_mass}" radius="${wheel_radius}" length="${wheel_thickness}">
-                <origin xyz="0.0 0.0 -${wheel_thickness/2}" rpy="0.0 0.0 0.0"/>
-            </xacro:inertial_cylinder>
+            <inertial>
+                <origin xyz="0.0 0.0 0.0" rpy="0.0 0.0 0.0"/>
+                <mass value="0.0064"/>
+                <inertia ixx="0.000046803"
+                         ixy="0.0"
+                         ixz="0.0"
+                         iyy="0.000046833"
+                         iyz="0.0"
+                         izz="0.000089214"/>
+            </inertial>
         </link>
+        <xacro:insert_roller parent="wheel${suffix}_link" reflect="1.0" theta="0" suffix="1" wheel="${suffix}"/>
+        <xacro:insert_roller parent="wheel${suffix}_link" reflect="1.0" theta="${PI/6}" suffix="2" wheel="${suffix}"/>
+        <xacro:insert_roller parent="wheel${suffix}_link" reflect="1.0" theta="${PI/3}" suffix="3" wheel="${suffix}"/>
+        <xacro:insert_roller parent="wheel${suffix}_link" reflect="1.0" theta="${PI/2}" suffix="4" wheel="${suffix}"/>
+        <xacro:insert_roller parent="wheel${suffix}_link" reflect="1.0" theta="${2*PI/3}" suffix="5" wheel="${suffix}"/>
+        <xacro:insert_roller parent="wheel${suffix}_link" reflect="1.0" theta="${5*PI/6}" suffix="6" wheel="${suffix}"/>
+        <xacro:insert_roller parent="wheel${suffix}_link" reflect="1.0" theta="${PI}" suffix="7" wheel="${suffix}"/>
+        <xacro:insert_roller parent="wheel${suffix}_link" reflect="1.0" theta="${7*PI/6}" suffix="8" wheel="${suffix}"/>
+        <xacro:insert_roller parent="wheel${suffix}_link" reflect="1.0" theta="${4*PI/3}" suffix="9" wheel="${suffix}"/>
+        <xacro:insert_roller parent="wheel${suffix}_link" reflect="1.0" theta="${3*PI/2}" suffix="10" wheel="${suffix}"/>
+        <xacro:insert_roller parent="wheel${suffix}_link" reflect="1.0" theta="${5*PI/3}" suffix="11" wheel="${suffix}"/>
+        <xacro:insert_roller parent="wheel${suffix}_link" reflect="1.0" theta="${11*PI/6}" suffix="12" wheel="${suffix}"/>
+        <xacro:insert_roller parent="wheel${suffix}_link" reflect="-1.0" theta="${45*PI/180}" suffix="-1" wheel="${suffix}"/>
+        <xacro:insert_roller parent="wheel${suffix}_link" reflect="-1.0" theta="${75*PI/180}" suffix="-2" wheel="${suffix}"/>
+        <xacro:insert_roller parent="wheel${suffix}_link" reflect="-1.0" theta="${105*PI/180}" suffix="-3" wheel="${suffix}"/>
+        <xacro:insert_roller parent="wheel${suffix}_link" reflect="-1.0" theta="${135*PI/180}" suffix="-4" wheel="${suffix}"/>
+        <xacro:insert_roller parent="wheel${suffix}_link" reflect="-1.0" theta="${165*PI/180}" suffix="-5" wheel="${suffix}"/>
+        <xacro:insert_roller parent="wheel${suffix}_link" reflect="-1.0" theta="${195*PI/180}" suffix="-6" wheel="${suffix}"/>
+        <xacro:insert_roller parent="wheel${suffix}_link" reflect="-1.0" theta="${225*PI/180}" suffix="-7" wheel="${suffix}"/>
+        <xacro:insert_roller parent="wheel${suffix}_link" reflect="-1.0" theta="${255*PI/180}" suffix="-8" wheel="${suffix}"/>
+        <xacro:insert_roller parent="wheel${suffix}_link" reflect="-1.0" theta="${285*PI/180}" suffix="-9" wheel="${suffix}"/>
+        <xacro:insert_roller parent="wheel${suffix}_link" reflect="-1.0" theta="${315*PI/180}" suffix="-10" wheel="${suffix}"/>
+        <xacro:insert_roller parent="wheel${suffix}_link" reflect="-1.0" theta="${345*PI/180}" suffix="-11" wheel="${suffix}"/>
+        <xacro:insert_roller parent="wheel${suffix}_link" reflect="-1.0" theta="${375*PI/180}" suffix="-12" wheel="${suffix}"/>
     </xacro:macro>
 </robot>
