Commit message: Add visual URDF blocks of wheels

File: axebot_description/urdf/axebot.urdf.xacro (robot description, xacro)
@@ -4,21 +4,3 @@
     <xacro:include filename="$(find axebot_description)/urdf/axebot_description.urdf.xacro"/>
     <xacro:axebot prefix="$(arg prefix)"/>
-  <!-- <link name="base_link">
-    <visual>
-      <geometry>
-        <cylinder length="0.6" radius="0.2"/>
-      </geometry>
-    </visual>
-  </link>
-  <link name="right_leg">
-    <visual>
-      <geometry>
-        <box size="0.6 0.1 0.2"/>
-      </geometry>
-    </visual>
-  </link>
-  <joint name="base_to_right_leg" type="fixed">
-    <parent link="base_link"/>
-    <child link="right_leg"/>
-  </joint> -->
 </robot>

File: axebot_description/urdf/axebot_description.urdf.xacro (robot description, xacro)
@@ -1,17 +1,22 @@
 <?xml version="1.0"?>
 <robot xmlns:xacro="http://www.ros.org/wiki/xacro">
+    <!-- Constants for wheel mechanical parameters -->
+    <xacro:property name="PI" value="3.1415926535897931"/>
+    <xacro:property name="base_mass" value="1.551"/>
+    <xacro:property name="base_height" value="0.04"/>
+    <xacro:property name="robot_height" value="0.053"/>
+    <xacro:property name="wheel_mass" value="0.3" />
+    <xacro:property name="wheel_radius" value="0.05" />
+    <xacro:property name="wheel_shaft_radius" value="0.005" />
+    <!-- The sum of the base radius, half of wheel thickness, and the shat
+    length must be equal the robot radius L = 0.1 m used in the kinematic model -->
+    <xacro:property name="base_radius" value="0.085"/>
+    <xacro:property name="wheel_thickness" value="0.025" />
+    <xacro:property name="distance_to_chassis" value="0.0025"/>
+    <xacro:include filename="$(find axebot_description)/urdf/axebot_wheels.urdf.xacro"/>
     <xacro:macro name="axebot" params="prefix">
-        <!-- Constants for robot dimensions -->
-        <xacro:property name="PI" value="3.1415926535897931"/>
-        <xacro:property name="base_mass" value="1.551" />
-        <xacro:property name="base_radius" value="0.1" />
-        <xacro:property name="base_height" value="0.02" />
-        <xacro:property name="wheel_mass" value="0.3" />
-        <xacro:property name="wheel_len" value="0.005" />
-        <xacro:property name="wheel_radius" value="0.015" />
-        <xacro:property name="z_offset" value="-${base_height/2}" />
         <link name="${prefix}base_link">
             <visual name="">
-                <origin xyz="0.0 0.0 ${base_height/2 + wheel_radius/2}" rpy="0.0 0.0 0.0"/>
+                <origin xyz="0.0 0.0 ${robot_height}" rpy="0.0 0.0 0.0"/>
                 <geometry>
                     <cylinder radius="${base_radius}" length="${base_height}"/>
@@ -20,18 +25,7 @@
             </visual>
         </link>
-        <joint name="${prefix}wheel1_joint" type="continuous">
-            <origin xyz="-${base_radius} 0.0 ${wheel_radius/2}" rpy="0.0 -${PI/2} 0.0"/>
-            <parent link="${prefix}base_link"/>
-            <child link="${prefix}wheel1_link"/>
-            <axis xyz="0.0 0.0 1.0"/>
-        </joint>
-        <link name="${prefix}wheel1_link">
-            <visual>
-                <origin xyz="0.0 0.0 ${wheel_len/2}" rpy="0.0 0.0 0.0"/>
-                <geometry>
-                    <cylinder radius="${wheel_radius}" length="${wheel_len}"/>
-                </geometry>
-            </visual>
-        </link>
+        <xacro:wheel prefix="${prefix}" num="1" theta="${PI}"/>
+        <xacro:wheel prefix="${prefix}" num="2" theta="-${PI/3}"/>
+        <xacro:wheel prefix="${prefix}" num="3" theta="${PI/3}"/>
     </xacro:macro>
 </robot>

Commit message: Remove unnecessary URDF file

File: axebot_description/urdf/axebot.urdf.xacro (robot description, xacro)
@@ -1,6 +1,42 @@
 <?xml version="1.0"?>
 <robot xmlns:xacro="http://www.ros.org/wiki/xacro" name="axebot">
+    <!-- Constants for wheel mechanical parameters -->
+    <xacro:property name="PI" value="3.1415926535897931"/>
+    <xacro:property name="base_mass" value="1.551"/>
+    <xacro:property name="base_height" value="0.04"/>
+    <xacro:property name="robot_height" value="0.053"/>
+    <xacro:property name="wheel_mass" value="0.268" />
+    <xacro:property name="wheel_radius" value="0.05" />
+    <xacro:property name="wheel_shaft_radius" value="0.005" />
+    <xacro:property name="shaft_mass" value="0.01" />
+    <!-- The sum of the base radius, half of wheel thickness, and the shat
+    length must be equal the robot radius L = 0.1 m used in the kinematic model -->
+    <xacro:property name="base_radius" value="0.085"/>
+    <xacro:property name="wheel_thickness" value="0.025" />
+    <xacro:property name="shaft_length" value="0.0025"/>
+    <xacro:include filename="$(find axebot_description)/urdf/wheel.urdf.xacro"/>
+    <xacro:include filename="$(find axebot_description)/urdf/materials.urdf.xacro"/>
     <xacro:arg name="prefix" default=""/>
-    <xacro:include filename="$(find axebot_description)/urdf/axebot_description.urdf.xacro"/>
-    <xacro:axebot prefix="$(arg prefix)"/>
+    <link name="$(arg prefix)base_link">
+        <visual name="">
+            <origin xyz="0.0 0.0 ${robot_height}" rpy="0.0 0.0 0.0"/>
+            <geometry>
+                <cylinder radius="${base_radius}" length="${base_height}"/>
+            </geometry>
+            <material name="black"/>
+        </visual>
+        <collision>
+            <origin xyz="0.0 0.0 ${robot_height}" rpy="0.0 0.0 0.0"/>
+            <geometry>
+                <cylinder radius="${base_radius}" length="${base_height}"/>
+            </geometry>
+            <material name="black"/>
+        </collision>
+        <xacro:inertial_cylinder mass="${base_mass}" radius="${base_radius}" length="${base_height}">
+            <origin xyz="0.0 0.0 ${robot_height}" rpy="0.0 0.0 0.0"/>
+        </xacro:inertial_cylinder>
+    </link>
+    <xacro:wheel prefix="$(arg prefix)" num="1" theta="${PI}"/>
+    <xacro:wheel prefix="$(arg prefix)" num="2" theta="-${PI/3}"/>
+    <xacro:wheel prefix="$(arg prefix)" num="3" theta="${PI/3}"/>
 </robot>

Commit message: Improve wheel xacro

File: axebot_description/urdf/axebot.urdf.xacro (robot description, xacro)
@@ -37,6 +37,6 @@
         </xacro:inertial_cylinder>
     </link>
-    <xacro:wheel prefix="$(arg prefix)" num="1" theta="${PI}"/>
-    <xacro:wheel prefix="$(arg prefix)" num="2" theta="-${PI/3}"/>
-    <xacro:wheel prefix="$(arg prefix)" num="3" theta="${PI/3}"/>
+    <xacro:wheel parent="$(arg prefix)base_link" suffix="1" theta="${PI}"/>
+    <xacro:wheel parent="$(arg prefix)base_link" suffix="2" theta="-${PI/3}"/>
+    <xacro:wheel parent="$(arg prefix)base_link" suffix="3" theta="${PI/3}"/>
 </robot>

File: axebot_description/urdf/wheel.urdf.xacro (robot description, xacro)
@@ -14,11 +14,11 @@
             </inertial>
     </xacro:macro>
-    <xacro:macro name="wheel" params="prefix num theta">
-        <joint name="${prefix}wheel${num}_shaft_joint" type="fixed">
+    <xacro:macro name="wheel" params="parent suffix theta">
+        <joint name="wheel${suffix}_shaft_joint" type="fixed">
             <origin xyz="${base_radius*cos(theta)} ${base_radius*sin(theta)} ${robot_height}" rpy="0.0 ${PI/2} ${theta+PI}"/>
-            <parent link="${prefix}base_link"/>
-            <child link="${prefix}wheel${num}_shaft_link"/>
+            <parent link="${parent}"/>
+            <child link="wheel${suffix}_shaft_link"/>
         </joint>
-        <link name="${prefix}wheel${num}_shaft_link">
+        <link name="wheel${suffix}_shaft_link">
             <visual>
                 <origin xyz="0.0 0.0 -${shaft_length/2}" rpy="0.0 0.0 0.0"/>
@@ -38,11 +38,11 @@
             </xacro:inertial_cylinder>
         </link>
-        <joint name="${prefix}wheel${num}_joint" type="continuous">
+        <joint name="wheel${suffix}_joint" type="continuous">
             <origin xyz="0.0 0.0 -${shaft_length}" rpy="0.0 0.0 0.0"/>
-            <parent link="${prefix}wheel${num}_shaft_link"/>
-            <child link="${prefix}wheel${num}_link"/>
+            <parent link="wheel${suffix}_shaft_link"/>
+            <child link="wheel${suffix}_link"/>
             <axis xyz="0.0 0.0 1.0"/>
         </joint>
-        <link name="${prefix}wheel${num}_link">
+        <link name="wheel${suffix}_link">
             <visual>
                 <origin xyz="0.0 0.0 -${wheel_thickness/2}" rpy="0.0 0.0 0.0"/>

Commit message: Improve shaft property and link naming

File: axebot_description/urdf/axebot.urdf.xacro (robot description, xacro)
@@ -8,5 +8,5 @@
     <xacro:property name="wheel_mass" value="0.268" />
     <xacro:property name="wheel_radius" value="0.05" />
-    <xacro:property name="wheel_shaft_radius" value="0.005" />
+    <xacro:property name="motor_shaft_radius" value="0.005" />
     <xacro:property name="shaft_mass" value="0.01" />
     <!-- The sum of the base radius, half of wheel thickness, and the shat
@@ -14,5 +14,5 @@
     <xacro:property name="base_radius" value="0.085"/>
     <xacro:property name="wheel_thickness" value="0.025" />
-    <xacro:property name="shaft_length" value="0.0025"/>
+    <xacro:property name="motor_shaft_length" value="0.0025"/>
     <xacro:include filename="$(find axebot_description)/urdf/wheel.urdf.xacro"/>
     <xacro:include filename="$(find axebot_description)/urdf/materials.urdf.xacro"/>

File: axebot_description/urdf/wheel.urdf.xacro (robot description, xacro)
@@ -18,27 +18,27 @@
             <origin xyz="${base_radius*cos(theta)} ${base_radius*sin(theta)} ${robot_height}" rpy="0.0 ${PI/2} ${theta+PI}"/>
             <parent link="${parent}"/>
-            <child link="wheel${suffix}_shaft_link"/>
+            <child link="motor${suffix}_shaft_link"/>
         </joint>
-        <link name="wheel${suffix}_shaft_link">
+        <link name="motor${suffix}_shaft_link">
             <visual>
-                <origin xyz="0.0 0.0 -${shaft_length/2}" rpy="0.0 0.0 0.0"/>
+                <origin xyz="0.0 0.0 -${motor_shaft_length/2}" rpy="0.0 0.0 0.0"/>
                 <geometry>
-                    <cylinder radius="${wheel_shaft_radius}" length="${shaft_length}"/>
+                    <cylinder radius="${motor_shaft_radius}" length="${motor_shaft_length}"/>
                 </geometry>
                 <material name="grey"/>
             </visual>
             <collision>
-                <origin xyz="0.0 0.0 -${shaft_length/2}" rpy="0.0 0.0 0.0"/>
+                <origin xyz="0.0 0.0 -${motor_shaft_length/2}" rpy="0.0 0.0 0.0"/>
                 <geometry>
-                    <cylinder radius="${wheel_shaft_radius}" length="${shaft_length}"/>
+                    <cylinder radius="${motor_shaft_radius}" length="${motor_shaft_length}"/>
                 </geometry>
             </collision>
-            <xacro:inertial_cylinder mass="${shaft_mass}" radius="${wheel_shaft_radius}" length="${shaft_length}">
-                <origin xyz="0.0 0.0 -${shaft_length/2}" rpy="0.0 0.0 0.0"/>
+            <xacro:inertial_cylinder mass="${shaft_mass}" radius="${motor_shaft_radius}" length="${motor_shaft_length}">
+                <origin xyz="0.0 0.0 -${motor_shaft_length/2}" rpy="0.0 0.0 0.0"/>
             </xacro:inertial_cylinder>
         </link>
         <joint name="wheel${suffix}_joint" type="continuous">
-            <origin xyz="0.0 0.0 -${shaft_length}" rpy="0.0 0.0 0.0"/>
-            <parent link="wheel${suffix}_shaft_link"/>
+            <origin xyz="0.0 0.0 -${motor_shaft_length}" rpy="0.0 0.0 0.0"/>
+            <parent link="motor${suffix}_shaft_link"/>
             <child link="wheel${suffix}_link"/>
             <axis xyz="0.0 0.0 1.0"/>

Commit message: Add chassis link

File: axebot_description/urdf/axebot.urdf.xacro (robot description, xacro)
@@ -3,6 +3,6 @@
     <!-- Constants for wheel mechanical parameters -->
     <xacro:property name="PI" value="3.1415926535897931"/>
-    <xacro:property name="base_mass" value="1.551"/>
-    <xacro:property name="base_height" value="0.04"/>
+    <xacro:property name="chassis_mass" value="1.551"/>
+    <xacro:property name="chassis_height" value="0.04"/>
     <xacro:property name="robot_height" value="0.053"/>
     <xacro:property name="wheel_mass" value="0.268" />
@@ -10,17 +10,22 @@
     <xacro:property name="motor_shaft_radius" value="0.005" />
     <xacro:property name="shaft_mass" value="0.01" />
-    <!-- The sum of the base radius, half of wheel thickness, and the shat
+    <!-- The sum of the chassis radius, half of wheel thickness, and the motor shaft
     length must be equal the robot radius L = 0.1 m used in the kinematic model -->
-    <xacro:property name="base_radius" value="0.085"/>
+    <xacro:property name="chassis_radius" value="0.085"/>
     <xacro:property name="wheel_thickness" value="0.025" />
     <xacro:property name="motor_shaft_length" value="0.0025"/>
     <xacro:include filename="$(find axebot_description)/urdf/wheel.urdf.xacro"/>
     <xacro:include filename="$(find axebot_description)/urdf/materials.urdf.xacro"/>
-    <xacro:arg name="prefix" default=""/>
-    <link name="$(arg prefix)base_link">
+    <link name="base_link"></link>
+    <joint name="base_link_joint" type="fixed">
+        <origin xyz="0 0 0" rpy="0 0 0" />
+        <parent link="base_link"/>
+        <child link="chassis_link" />
+    </joint>
+    <link name="chassis_link">
         <visual name="">
             <origin xyz="0.0 0.0 ${robot_height}" rpy="0.0 0.0 0.0"/>
             <geometry>
-                <cylinder radius="${base_radius}" length="${base_height}"/>
+                <cylinder radius="${chassis_radius}" length="${chassis_height}"/>
             </geometry>
             <material name="black"/>
@@ -29,14 +34,14 @@
             <origin xyz="0.0 0.0 ${robot_height}" rpy="0.0 0.0 0.0"/>
             <geometry>
-                <cylinder radius="${base_radius}" length="${base_height}"/>
+                <cylinder radius="${chassis_radius}" length="${chassis_height}"/>
             </geometry>
             <material name="black"/>
         </collision>
-        <xacro:inertial_cylinder mass="${base_mass}" radius="${base_radius}" length="${base_height}">
+        <xacro:inertial_cylinder mass="${chassis_mass}" radius="${chassis_radius}" length="${chassis_height}">
             <origin xyz="0.0 0.0 ${robot_height}" rpy="0.0 0.0 0.0"/>
         </xacro:inertial_cylinder>
     </link>
-    <xacro:wheel parent="$(arg prefix)base_link" suffix="1" theta="${PI}"/>
-    <xacro:wheel parent="$(arg prefix)base_link" suffix="2" theta="-${PI/3}"/>
-    <xacro:wheel parent="$(arg prefix)base_link" suffix="3" theta="${PI/3}"/>
+    <xacro:wheel parent="chassis_link" suffix="1" theta="${PI}"/>
+    <xacro:wheel parent="chassis_link" suffix="2" theta="-${PI/3}"/>
+    <xacro:wheel parent="chassis_link" suffix="3" theta="${PI/3}"/>
 </robot>

File: axebot_description/urdf/wheel.urdf.xacro (robot description, xacro)
@@ -16,5 +16,5 @@
     <xacro:macro name="wheel" params="parent suffix theta">
         <joint name="wheel${suffix}_shaft_joint" type="fixed">
-            <origin xyz="${base_radius*cos(theta)} ${base_radius*sin(theta)} ${robot_height}" rpy="0.0 ${PI/2} ${theta+PI}"/>
+            <origin xyz="${chassis_radius*cos(theta)} ${chassis_radius*sin(theta)} ${robot_height}" rpy="0.0 ${PI/2} ${theta+PI}"/>
             <parent link="${parent}"/>
             <child link="motor${suffix}_shaft_link"/>

Commit message: Update real robot physics parameters

File: axebot_description/urdf/axebot.urdf.xacro (robot description, xacro)
@@ -3,13 +3,14 @@
     <!-- Constants for wheel mechanical parameters -->
     <xacro:property name="PI" value="3.1415926535897931"/>
-    <xacro:property name="chassis_mass" value="1.551"/>
+    <xacro:property name="chassis_mass" value="1.074"/>
     <xacro:property name="chassis_height" value="0.04"/>
     <xacro:property name="robot_height" value="0.053"/>
-    <xacro:property name="wheel_mass" value="0.268" />
-    <xacro:property name="wheel_radius" value="0.05" />
-    <xacro:property name="motor_shaft_radius" value="0.005" />
-    <xacro:property name="shaft_mass" value="0.01" />
-    <!-- The sum of the chassis radius, half of wheel thickness, and the motor shaft
-    length must be equal the robot radius L = 0.1 m used in the kinematic model -->
+    <xacro:property name="wheel_mass" value="0.105" />
+    <xacro:property name="wheel_radius" value="0.0508" />
+    <xacro:property name="motor_shaft_radius" value="0.002" />
+    <xacro:property name="shaft_mass" value="0.001" />
+    <!-- The sum of the chassis radius, half the wheel thickness, and the
+    motor shaft length must be equal to the robot radius L = 0.1 m used in the
+    kinematic model -->
     <xacro:property name="chassis_radius" value="0.085"/>
     <xacro:property name="wheel_thickness" value="0.025" />
