Commit message: Update URDF with more realistic parameters - Parameters gathered in onshape software

File: axebot_description/urdf/axebot.urdf.xacro (robot description, xacro)
@@ -15,6 +15,6 @@
     kinematic model -->
     <xacro:property name="chassis_radius" value="0.085"/>
-    <xacro:property name="wheel_thickness" value="0.025" />
-    <xacro:property name="motor_shaft_length" value="0.0025"/>
+    <xacro:property name="wheel_thickness" value="0.01905" />
+    <xacro:property name="motor_shaft_length" value="0.005475"/>
     <xacro:include filename="$(find axebot_description)/urdf/wheel.urdf.xacro"/>
     <xacro:include filename="$(find axebot_description)/urdf/materials.urdf.xacro"/>
@@ -23,5 +23,5 @@
     <link name="base_link"></link>
     <joint name="base_link_joint" type="fixed">
-        <origin xyz="0 0 0" rpy="0 0 0" />
+        <origin xyz="0 0 ${robot_height}" rpy="0 0 0" />
         <parent link="base_link"/>
         <child link="chassis_link" />
@@ -29,5 +29,5 @@
     <link name="chassis_link">
         <visual name="">
-            <origin xyz="0.0 0.0 ${robot_height}" rpy="0.0 0.0 0.0"/>
+            <origin xyz="0.0 0.0 0.0" rpy="0.0 0.0 0.0"/>
             <geometry>
                 <cylinder radius="${chassis_radius}" length="${chassis_height}"/>
@@ -36,5 +36,5 @@
         </visual>
         <collision>
-            <origin xyz="0.0 0.0 ${robot_height}" rpy="0.0 0.0 0.0"/>
+            <origin xyz="0.0 0.0 0.0" rpy="0.0 0.0 0.0"/>
             <geometry>
                 <cylinder radius="${chassis_radius}" length="${chassis_height}"/>
@@ -42,7 +42,14 @@
             <material name="black"/>
         </collision>
-        <xacro:inertial_cylinder mass="${chassis_mass}" radius="${chassis_radius}" length="${chassis_height}">
-            <origin xyz="0.0 0.0 ${robot_height}" rpy="0.0 0.0 0.0"/>
-        </xacro:inertial_cylinder>
+        <inertial>
+            <origin xyz="0.0 0.0 0.0" rpy="0.0 0.0 0.0"/>
+            <mass value="1.634"/>
+            <inertia ixx="0.00316977667"
+                        ixy="0.0"
+                        ixz="0.0"
+                        iyy="0.00316977667"
+                        iyz="0.0"
+                        izz="0.005903752"/>
+        </inertial>
     </link>
     <xacro:if value="$(arg only_one_wheel)">

File: axebot_description/urdf/gazebo.urdf.xacro (robot description, xacro)
@@ -5,23 +5,34 @@
     <gazebo reference="wheel1_link">
         <material>Gazebo/Grey</material>
-        <mu1>1.2</mu1>
-        <mu2>1.2</mu2>
+        <!-- <fdir1>0 1 0"</fdir1> -->
+        <!-- <mu1>1.7</mu1> -->
+        <!-- <mu2>0.2</mu2> -->
     </gazebo>
     <gazebo reference="wheel2_link">
         <material>Gazebo/Grey</material>
-        <mu1>1.2</mu1>
-        <mu2>1.2</mu2>
+        <!-- <fdir1>0 1 0"</fdir1> -->
+        <!-- <mu1>1.7</mu1> -->
+        <!-- <mu2>0.2</mu2> -->
     </gazebo>
     <gazebo reference="wheel3_link">
         <material>Gazebo/Grey</material>
-        <mu1>1.2</mu1>
-        <mu2>1.2</mu2>
+        <!-- <fdir1>0 1 0"</fdir1> -->
+        <!-- <mu1>1.7</mu1> -->
+        <!-- <mu2>0.2</mu2> -->
     </gazebo>
     <gazebo>
         <plugin filename="libgazebo_ros2_control.so" name="gazebo_ros2_control">
-        <robot_param>robot_description</robot_param>
-        <robot_param_node>robot_state_publisher</robot_param_node>
-        <parameters>$(find axebot_control)/config/omnidirectional_controller.yaml</parameters>
-        <!-- <parameters>$(find axebot_description)/config/ros2_controllers.yaml</parameters> -->
+            <robot_param>robot_description</robot_param>
+            <robot_param_node>robot_state_publisher</robot_param_node>
+            <parameters>$(find axebot_control)/config/omnidirectional_controller.yaml</parameters>
+        </plugin>
+        <plugin filename="libgazebo_ros_p3d.so" name="gazebo_ros_p3d" >
+            <ros>
+                <namespace>ground_truth_odom</namespace>
+            </ros>
+            <frame_name>world</frame_name>
+            <body_name>base_link</body_name>
+            <update_rate>50.0</update_rate>
+            <gaussian_noise>0.01</gaussian_noise>
         </plugin>
     </gazebo>

File: axebot_description/urdf/materials.urdf.xacro (robot description, xacro)
@@ -9,3 +9,6 @@
     <color rgba="0.2 0.2 0.2 1.0"/>
   </material>
+  <material name="red">
+    <color rgba="1.0 0.0 0.0 1.0"/>
+  </material>
 </robot>

File: axebot_description/urdf/wheel.urdf.xacro (robot description, xacro)
@@ -16,9 +16,10 @@
     </xacro:macro>
     <xacro:macro name="insert_roller" params="parent reflect theta suffix wheel">
-        <joint name="rim_to_roller${wheel}${suffix}joint" type="fixed">
+        <joint name="rim_to_roller${wheel}${suffix}joint" type="continuous">
             <origin xyz="${distance_to_roller_center*cos(theta)} ${distance_to_roller_center*sin(theta)} ${reflect*0.008}" rpy="0.0 0.0 ${theta-PI/2}"/>
             <parent link="${parent}"/>
             <child link="roller${wheel}${suffix}_link"/>
             <axis xyz="1.0 0.0 0.0"/>
+            <dynamics friction="0.01"/>
         </joint>
         <link name="roller${wheel}${suffix}_link">
@@ -42,13 +43,19 @@
                          ixy="0.0"
                          ixz="0.0"
-                         iyy="7.6e-8"
+                         iyy="8e-8"
                          iyz="0.0"
-                         izz="7.6e-8"/>
+                         izz="8e-8"/>
             </inertial>
         </link>
+        <gazebo reference="roller${wheel}${suffix}_link">
+            <material>Gazebo/Green</material>
+            <fdir1>0 1 0"</fdir1>
+            <mu1>10</mu1>
+            <mu2>10</mu2>
+        </gazebo>
     </xacro:macro>
     <xacro:macro name="wheel" params="parent suffix theta">
         <joint name="wheel${suffix}_shaft_joint" type="fixed">
-            <origin xyz="${chassis_radius*cos(theta)} ${chassis_radius*sin(theta)} ${robot_height}" rpy="0.0 ${PI/2} ${theta+PI}"/>
+            <origin xyz="${chassis_radius*cos(theta)} ${chassis_radius*sin(theta)} 0.0" rpy="0.0 ${PI/2} ${theta+PI}"/>
             <parent link="${parent}"/>
             <child link="motor${suffix}_shaft_link"/>
@@ -60,5 +67,5 @@
                     <cylinder radius="${motor_shaft_radius}" length="${motor_shaft_length}"/>
                 </geometry>
-                <material name="grey"/>
+                <material name="red"/>
             </visual>
             <collision>
@@ -73,5 +80,5 @@
         </link>
         <joint name="wheel${suffix}_joint" type="continuous">
-            <origin xyz="0.0 0.0 -${motor_shaft_length}" rpy="0.0 0.0 0.0"/>
+            <origin xyz="0.0 0.0 -${motor_shaft_length+wheel_thickness/2}" rpy="0.0 0.0 0.0"/>
             <parent link="motor${suffix}_shaft_link"/>
             <child link="wheel${suffix}_link"/>
@@ -87,18 +94,18 @@
             </visual>
             <collision>
-                <origin xyz="0.0 0.0 -${wheel_thickness/2}" rpy="0.0 0.0 0.0"/>
+                <origin xyz="0.0 0.0 0.0" rpy="0.0 0.0 0.0"/>
                 <geometry>
-                    <mesh filename="file://$(find axebot_description)/meshes/rim.stl"/>
+                    <mesh filename="file://$(find axebot_description)/meshes/wheel-collision.dae"/>
                 </geometry>
             </collision>
             <inertial>
                 <origin xyz="0.0 0.0 0.0" rpy="0.0 0.0 0.0"/>
-                <mass value="0.0064"/>
-                <inertia ixx="0.000046803"
+                <mass value="0.113"/>
+                <inertia ixx="0.000089064"
                          ixy="0.0"
                          ixz="0.0"
-                         iyy="0.000046833"
+                         iyy="0.000089064"
                          iyz="0.0"
-                         izz="0.000089214"/>
+                         izz="0.000173339"/>
             </inertial>
         </link>
