Commit message: Add rim mesh to collision in omni wheels

File: axebot_description/urdf/wheel.urdf.xacro (robot description, xacro)
@@ -89,5 +89,5 @@
                 <origin xyz="0.0 0.0 -${wheel_thickness/2}" rpy="0.0 0.0 0.0"/>
                 <geometry>
-                    <cylinder radius="${wheel_radius}" length="${wheel_thickness}"/>
+                    <mesh filename="file://$(find axebot_description)/meshes/rim.stl"/>
                 </geometry>
             </collision>

Commit message: Improve friction parameters of omni wheels

File: axebot_description/urdf/wheel.urdf.xacro (robot description, xacro)
@@ -21,5 +21,5 @@
             <child link="roller${wheel}${suffix}_link"/>
             <axis xyz="1.0 0.0 0.0"/>
-            <dynamics friction="0.01"/>
+            <dynamics friction="0.1"/>
         </joint>
         <link name="roller${wheel}${suffix}_link">
@@ -50,7 +50,8 @@
         <gazebo reference="roller${wheel}${suffix}_link">
             <material>Gazebo/Green</material>
-            <fdir1>0 1 0"</fdir1>
-            <mu1>10</mu1>
-            <mu2>10</mu2>
+            <fdir1>1 0 0"</fdir1>
+            <mu1>100</mu1>
+            <mu2>100</mu2>
+            <minDepth>0.001</minDepth>
         </gazebo>
     </xacro:macro>
